Commit message: Change launch and rviz config

File: jetbot_mirea_description/urdf/jetbot_mirea.urdf.xacro (robot description, xacro)
@@ -234,5 +234,5 @@
     <parent link="base_link"/>
     <child link="rplidar_link"/>
-    <origin xyz="0.087 0.0 -0.003" rpy="3.14 0.0 0.0"/>
+    <origin xyz="0.087 0.0 -0.003" rpy="3.14 0.0 2.3562"/>
   </joint>
   <link name="rplidar_link">
